Commit message: M7 doneeeeeeeeeeeeeeeeeeeee

File: urdf/mounted_ur.urdf.xacro (robot description, xacro)
@@ -50,5 +50,28 @@
     parent="$(arg prefix)tool0"
     sim_ignition="$(arg sim_ignition)"/>
+  <!-- Fortress fixed-joint constraints for the Assignment 03 physical grasp.
+       Gazebo merges gripper_base's fixed joint into wrist_3_link, so the
+       surviving wrist link is the physical parent. Each cube's SDF link is
+       named link. The M7 manager detaches initial joints before any motion. -->
+  <xacro:macro name="assignment_cube_joint" params="cube">
+    <gazebo>
+      <plugin filename="ignition-gazebo-detachable-joint-system"
+              name="ignition::gazebo::systems::DetachableJoint">
+        <parent_link>wrist_3_link</parent_link>
+        <child_model>${cube}</child_model>
+        <child_link>link</child_link>
+        <detach_topic>/m7/grasp/${cube}/detach</detach_topic>
+        <attach_topic>/m7/grasp/${cube}/attach</attach_topic>
+        <output_topic>/m7/grasp/${cube}/state</output_topic>
+        <suppress_child_warning>true</suppress_child_warning>
+      </plugin>
+    </gazebo>
+  </xacro:macro>
   <xacro:if value="$(arg sim_ignition)">
+    <xacro:assignment_cube_joint cube="red_cube"/>
+    <xacro:assignment_cube_joint cube="yellow_cube"/>
+    <xacro:assignment_cube_joint cube="blue_cube"/>
+    <xacro:assignment_cube_joint cube="green_cube"/>
+    <xacro:assignment_cube_joint cube="purple_cube"/>
     <gazebo reference="world"/>
     <gazebo>
